File: pcb/incinerator/incinerator.sch (KiCad schematic (older format))
At the start: 3 parts

Commit message: Completed schematic
Parts:
- added BZ1: Buzzer, symbol Device:Buzzer
- added C1: 0.33, symbol Device:CP
- added D1: DIODE, symbol pspice:DIODE
- added D2, D3, D4, D5, D6, D7: LED, symbol Device:LED
- added J1: Furnace Control, symbol Connector:Conn_01x06_Male
- added J5, J6: Adafruit MAX31855, symbol Connector:Conn_01x06_Female
- added R1: 200K, symbol Device:R
- added R2: 300K, symbol Device:R
- added R3, R4, R5, R6, R7, R8: 50, symbol Device:R
- added SW1: Rotary_Encoder_Switch, symbol Device:Rotary_Encoder_Switch
- gave numbers to parts that had none: 3
Connections:
- net GND is gone; now on net Earth: J3.2 (Pin_2), J4.7 (Pin_7)
- net 3V3: now also J5.1 (Pin_1), J6.1 (Pin_1)
- net D12: now also J2.4 (Pin_4), SW1.B
- net D13: now also J2.3 (Pin_3), SW1.A
- net D14: now also J2.5 (Pin_5), J1.6 (Pin_6), R3.1
- net D15: now also J3.3 (Pin_3), SW1.S1
- net D18: now also J5.6 (Pin_6), J6.6 (Pin_6)
- net D19: now also J5.4 (Pin_4), J6.4 (Pin_4); no longer J4.3 (Pin_3)
- net D22: now also J3.14 (Pin_14), BZ1.1 (-)
- net D25: now also J2.8 (Pin_8), J1.3 (Pin_3), R6.1
- net D26: now also J2.7 (Pin_7), J1.4 (Pin_4), R5.1
- net D27: now also J2.6 (Pin_6), J1.5 (Pin_5), R4.1
- net D32: now also J2.10 (Pin_10), J1.1 (Pin_1), R8.1
- net D33: now also J2.9 (Pin_9), J1.2 (Pin_2), R7.1
- net D4: now also J3.5 (Pin_5), J6.5 (Pin_5)
- net RX2: now also J3.6 (Pin_6), J5.5 (Pin_5)
- net TX2: now also J3.7 (Pin_7), J4.3 (Pin_3)
- net VIN: now also J2.1 (Pin_1), C1.1, D1.2 (A)
- net VN: now also J2.13 (Pin_13), R1.2, R2.1
- net Earth: now reaches J2.2 (Pin_2)
- net Earth: now also BZ1.2 (+), C1.2, D2.1 (K), D3.1 (K), D4.1 (K), D5.1 (K), D6.1 (K), D7.1 (K), J5.3 (Pin_3), J6.3 (Pin_3), R2.2, SW1.C, SW1.S2
- new net: D7.2 (A), R8.2
- new net: D6.2 (A), R7.2
- new net: D5.2 (A), R6.2
- new net: D4.2 (A), R5.2
- new net: D3.2 (A), R4.2
- new net: D2.2 (A), R3.2
- new net +5V: D1.1 (K), R1.1
Other:
- moved on the sheet: J2, J3, J4
