File: pcb/incinerator.sch (KiCad schematic (older format))
At the start: 51 parts, among them J1 Power Source 12V, J2 IGNITION_MAIN, J3 IGNITION_AFT, J4 VALVE_MAIN, J5 VALVE_AFT_HI, J6 VALVE_AFT_LO, J7 AIRPMP, J8 To Rotary Encoder / Switch, J9 Waveshare 4.2\" e-paper, Q1 IRLU120N, Q2 IRLU120N, Q3 IRLU120N, Q4 IRLU120N, Q5 IRLU120N, Q6 IRLU120N, U1 R-7890-0.5, U2 NodeMCU_ESP32, U3 Adafruit_MAX31855, U4 Adafruit_MAX31855

Commit message: reduced THT footprints from 10.16 to 7.62mm
Parts:
- D1, D11, D2, D4, D6, D9: footprint Diode_THT:D_DO-41_SOD81_P10.16mm_Horizontal -> Diode_THT:D_DO-41_SOD81_P7.62mm_Horizontal
- R1, R10, R11, R12, R13, R14, R15, R16, R17, R18, R2, R3, R4, R5, R6, R7, R8, R9: footprint Resistor_THT:R_Axial_DIN0207_L6.3mm_D2.5mm_P10.16mm_Horizontal -> Resistor_THT:R_Axial_DIN0207_L6.3mm_D2.5mm_P7.62mm_Horizontal
Changed lines of the file:
@@
 F 0 "R13" V 5107 1550 50  0000 C CNN
 F 1 "100" V 5016 1550 50  0000 C CNN
-F 2 "Resistor_THT:R_Axial_DIN0207_L6.3mm_D2.5mm_P10.16mm_Horizontal" V 4830 1550 50  0001 C CNN
+F 2 "Resistor_THT:R_Axial_DIN0207_L6.3mm_D2.5mm_P7.62mm_Horizontal" V 4830 1550 50  0001 C CNN
 F 3 "~" H 4900 1550 50  0001 C CNN
 	1    4900 1550
@@
 F 0 "R7" V 4657 1750 50  0000 C CNN
 F 1 "15k" V 4566 1750 50  0000 C CNN
-F 2 "Resistor_THT:R_Axial_DIN0207_L6.3mm_D2.5mm_P10.16mm_Horizontal" V 4380 1750 50  0001 C CNN
+F 2 "Resistor_THT:R_Axial_DIN0207_L6.3mm_D2.5mm_P7.62mm_Horizontal" V 4380 1750 50  0001 C CNN
 F 3 "~" H 4450 1750 50  0001 C CNN
 	1    4450 1750
@@
 F 0 "D1" V 2804 1679 50  0000 L CNN
 F 1 "D" V 2895 1679 50  0000 L CNN
-F 2 "Diode_THT:D_DO-41_SOD81_P10.16mm_Horizontal" H 2850 1600 50  0001 C CNN
+F 2 "Diode_THT:D_DO-41_SOD81_P7.62mm_Horizontal" H 2850 1600 50  0001 C CNN
 F 3 "~" H 2850 1600 50  0001 C CNN
 	1    2850 1600
@@
 F 0 "R1" V 2943 1450 50  0000 C CNN
 F 1 "1k" V 3034 1450 50  0000 C CNN
-F 2 "Resistor_THT:R_Axial_DIN0207_L6.3mm_D2.5mm_P10.16mm_Horizontal" V 3080 1450 50  0001 C CNN
+F 2 "Resistor_THT:R_Axial_DIN0207_L6.3mm_D2.5mm_P7.62mm_Horizontal" V 3080 1450 50  0001 C CNN
 F 3 "~" H 3150 1450 50  0001 C CNN
 	1    3150 1450
@@
 F 0 "R4" V 5107 2250 50  0000 C CNN
 F 1 "100" V 5016 2250 50  0000 C CNN
-F 2 "Resistor_THT:R_Axial_DIN0207_L6.3mm_D2.5mm_P10.16mm_Horizontal" V 4830 2250 50  0001 C CNN
+F 2 "Resistor_THT:R_Axial_DIN0207_L6.3mm_D2.5mm_P7.62mm_Horizontal" V 4830 2250 50  0001 C CNN
 F 3 "~" H 4900 2250 50  0001 C CNN
 	1    4900 2250
@@
 F 0 "R3" V 4657 2450 50  0000 C CNN
 F 1 "15k" V 4566 2450 50  0000 C CNN
-F 2 "Resistor_THT:R_Axial_DIN0207_L6.3mm_D2.5mm_P10.16mm_Horizontal" V 4380 2450 50  0001 C CNN
+F 2 "Resistor_THT:R_Axial_DIN0207_L6.3mm_D2.5mm_P7.62mm_Horizontal" V 4380 2450 50  0001 C CNN
 F 3 "~" H 4450 2450 50  0001 C CNN
 	1    4450 2450
@@
 F 0 "D2" V 2804 2379 50  0000 L CNN
 F 1 "D" V 2895 2379 50  0000 L CNN
-F 2 "Diode_THT:D_DO-41_SOD81_P10.16mm_Horizontal" H 2850 2300 50  0001 C CNN
+F 2 "Diode_THT:D_DO-41_SOD81_P7.62mm_Horizontal" H 2850 2300 50  0001 C CNN
 F 3 "~" H 2850 2300 50  0001 C CNN
 	1    2850 2300
@@
 F 0 "R2" V 2943 2150 50  0000 C CNN
 F 1 "1k" V 3034 2150 50  0000 C CNN
-F 2 "Resistor_THT:R_Axial_DIN0207_L6.3mm_D2.5mm_P10.16mm_Horizontal" V 3080 2150 50  0001 C CNN
+F 2 "Resistor_THT:R_Axial_DIN0207_L6.3mm_D2.5mm_P7.62mm_Horizontal" V 3080 2150 50  0001 C CNN
 F 3 "~" H 3150 2150 50  0001 C CNN
 	1    3150 2150
@@
 F 0 "R8" V 5107 2950 50  0000 C CNN
 F 1 "100" V 5016 2950 50  0000 C CNN
-F 2 "Resistor_THT:R_Axial_DIN0207_L6.3mm_D2.5mm_P10.16mm_Horizontal" V 4830 2950 50  0001 C CNN
+F 2 "Resistor_THT:R_Axial_DIN0207_L6.3mm_D2.5mm_P7.62mm_Horizontal" V 4830 2950 50  0001 C CNN
 F 3 "~" H 4900 2950 50  0001 C CNN
 	1    4900 2950
@@
 F 0 "R6" V 4657 3150 50  0000 C CNN
 F 1 "15k" V 4566 3150 50  0000 C CNN
-F 2 "Resistor_THT:R_Axial_DIN0207_L6.3mm_D2.5mm_P10.16mm_Horizontal" V 4380 3150 50  0001 C CNN
+F 2 "Resistor_THT:R_Axial_DIN0207_L6.3mm_D2.5mm_P7.62mm_Horizontal" V 4380 3150 50  0001 C CNN
 F 3 "~" H 4450 3150 50  0001 C CNN
 	1    4450 3150
@@
 F 0 "D4" V 2804 3079 50  0000 L CNN
 F 1 "D" V 2895 3079 50  0000 L CNN
-F 2 "Diode_THT:D_DO-41_SOD81_P10.16mm_Horizontal" H 2850 3000 50  0001 C CNN
+F 2 "Diode_THT:D_DO-41_SOD81_P7.62mm_Horizontal" H 2850 3000 50  0001 C CNN
 F 3 "~" H 2850 3000 50  0001 C CNN
 	1    2850 3000
@@
 F 0 "R5" V 2943 2850 50  0000 C CNN
 F 1 "1k" V 3034 2850 50  0000 C CNN
-F 2 "Resistor_THT:R_Axial_DIN0207_L6.3mm_D2.5mm_P10.16mm_Horizontal" V 3080 2850 50  0001 C CNN
+F 2 "Resistor_THT:R_Axial_DIN0207_L6.3mm_D2.5mm_P7.62mm_Horizontal" V 3080 2850 50  0001 C CNN
 F 3 "~" H 3150 2850 50  0001 C CNN
 	1    3150 2850
@@
 F 0 "R11" V 5107 3650 50  0000 C CNN
 F 1 "100" V 5016 3650 50  0000 C CNN
-F 2 "Resistor_THT:R_Axial_DIN0207_L6.3mm_D2.5mm_P10.16mm_Horizontal" V 4830 3650 50  0001 C CNN
+F 2 "Resistor_THT:R_Axial_DIN0207_L6.3mm_D2.5mm_P7.62mm_Horizontal" V 4830 3650 50  0001 C CNN
 F 3 "~" H 4900 3650 50  0001 C CNN
 	1    4900 3650
@@
 F 0 "R10" V 4657 3850 50  0000 C CNN
 F 1 "15k" V 4566 3850 50  0000 C CNN
-F 2 "Resistor_THT:R_Axial_DIN0207_L6.3mm_D2.5mm_P10.16mm_Horizontal" V 4380 3850 50  0001 C CNN
+F 2 "Resistor_THT:R_Axial_DIN0207_L6.3mm_D2.5mm_P7.62mm_Horizontal" V 4380 3850 50  0001 C CNN
 F 3 "~" H 4450 3850 50  0001 C CNN
 	1    4450 3850
@@
 F 0 "D6" V 2804 3779 50  0000 L CNN
 F 1 "D" V 2895 3779 50  0000 L CNN
-F 2 "Diode_THT:D_DO-41_SOD81_P10.16mm_Horizontal" H 2850 3700 50  0001 C CNN
+F 2 "Diode_THT:D_DO-41_SOD81_P7.62mm_Horizontal" H 2850 3700 50  0001 C CNN
 F 3 "~" H 2850 3700 50  0001 C CNN
 	1    2850 3700
@@
 F 0 "R9" V 2943 3550 50  0000 C CNN
 F 1 "1k" V 3034 3550 50  0000 C CNN
-F 2 "Resistor_THT:R_Axial_DIN0207_L6.3mm_D2.5mm_P10.16mm_Horizontal" V 3080 3550 50  0001 C CNN
+F 2 "Resistor_THT:R_Axial_DIN0207_L6.3mm_D2.5mm_P7.62mm_Horizontal" V 3080 3550 50  0001 C CNN
 F 3 "~" H 3150 3550 50  0001 C CNN
 	1    3150 3550
@@
 F 0 "R15" V 5107 4350 50  0000 C CNN
 F 1 "100" V 5016 4350 50  0000 C CNN
-F 2 "Resistor_THT:R_Axial_DIN0207_L6.3mm_D2.5mm_P10.16mm_Horizontal" V 4830 4350 50  0001 C CNN
+F 2 "Resistor_THT:R_Axial_DIN0207_L6.3mm_D2.5mm_P7.62mm_Horizontal" V 4830 4350 50  0001 C CNN
 F 3 "~" H 4900 4350 50  0001 C CNN
 	1    4900 4350
@@
 F 0 "R14" V 4657 4550 50  0000 C CNN
 F 1 "15k" V 4566 4550 50  0000 C CNN
-F 2 "Resistor_THT:R_Axial_DIN0207_L6.3mm_D2.5mm_P10.16mm_Horizontal" V 4380 4550 50  0001 C CNN
+F 2 "Resistor_THT:R_Axial_DIN0207_L6.3mm_D2.5mm_P7.62mm_Horizontal" V 4380 4550 50  0001 C CNN
 F 3 "~" H 4450 4550 50  0001 C CNN
 	1    4450 4550
@@
 F 0 "D9" V 2804 4479 50  0000 L CNN
 F 1 "D" V 2895 4479 50  0000 L CNN
-F 2 "Diode_THT:D_DO-41_SOD81_P10.16mm_Horizontal" H 2850 4400 50  0001 C CNN
+F 2 "Diode_THT:D_DO-41_SOD81_P7.62mm_Horizontal" H 2850 4400 50  0001 C CNN
 F 3 "~" H 2850 4400 50  0001 C CNN
 	1    2850 4400
@@
 F 0 "R12" V 2943 4250 50  0000 C CNN
 F 1 "1k" V 3034 4250 50  0000 C CNN
-F 2 "Resistor_THT:R_Axial_DIN0207_L6.3mm_D2.5mm_P10.16mm_Horizontal" V 3080 4250 50  0001 C CNN
+F 2 "Resistor_THT:R_Axial_DIN0207_L6.3mm_D2.5mm_P7.62mm_Horizontal" V 3080 4250 50  0001 C CNN
 F 3 "~" H 3150 4250 50  0001 C CNN
 	1    3150 4250
@@
 F 0 "R18" V 5107 5050 50  0000 C CNN
 F 1 "100" V 5016 5050 50  0000 C CNN
-F 2 "Resistor_THT:R_Axial_DIN0207_L6.3mm_D2.5mm_P10.16mm_Horizontal" V 4830 5050 50  0001 C CNN
+F 2 "Resistor_THT:R_Axial_DIN0207_L6.3mm_D2.5mm_P7.62mm_Horizontal" V 4830 5050 50  0001 C CNN
 F 3 "~" H 4900 5050 50  0001 C CNN
 	1    4900 5050
@@
 F 0 "R17" V 4657 5250 50  0000 C CNN
 F 1 "15k" V 4566 5250 50  0000 C CNN
-F 2 "Resistor_THT:R_Axial_DIN0207_L6.3mm_D2.5mm_P10.16mm_Horizontal" V 4380 5250 50  0001 C CNN
+F 2 "Resistor_THT:R_Axial_DIN0207_L6.3mm_D2.5mm_P7.62mm_Horizontal" V 4380 5250 50  0001 C CNN
 F 3 "~" H 4450 5250 50  0001 C CNN
 	1    4450 5250
@@
 F 0 "D11" V 2804 5179 50  0000 L CNN
 F 1 "D" V 2895 5179 50  0000 L CNN
-F 2 "Diode_THT:D_DO-41_SOD81_P10.16mm_Horizontal" H 2850 5100 50  0001 C CNN
+F 2 "Diode_THT:D_DO-41_SOD81_P7.62mm_Horizontal" H 2850 5100 50  0001 C CNN
 F 3 "~" H 2850 5100 50  0001 C CNN
 	1    2850 5100
@@
 F 0 "R16" V 2943 4950 50  0000 C CNN
 F 1 "1k" V 3034 4950 50  0000 C CNN
-F 2 "Resistor_THT:R_Axial_DIN0207_L6.3mm_D2.5mm_P10.16mm_Horizontal" V 3080 4950 50  0001 C CNN
+F 2 "Resistor_THT:R_Axial_DIN0207_L6.3mm_D2.5mm_P7.62mm_Horizontal" V 3080 4950 50  0001 C CNN
 F 3 "~" H 3150 4950 50  0001 C CNN
 	1    3150 4950

Commit message: re-worked & shrinked PCB
Parts:
- BZ1: footprint incinerator:Buzzer_BM_15B -> Buzzer_Beeper:Buzzer_TDK_PS1240P02BT_D12.2mm_H6.5mm
- D1, D11, D2, D4, D6, D9: footprint Diode_THT:D_DO-41_SOD81_P7.62mm_Horizontal -> incinerator:D_DO-41_P7.62mm_Custom
- D10, D12, D3, D5, D7, D8: footprint LED_THT:LED_D3.0mm -> incinerator:LED_D3.0mm_Custom
- Q1, Q2, Q3, Q4, Q5, Q6: footprint Package_TO_SOT_THT:SIPAK_Vertical -> incinerator:SIPAK_Vertical_Custom
- R1, R10, R11, R12, R13, R14, R15, R16, R17, R18, R2, R3, R4, R5, R6, R7, R8, R9: footprint Resistor_THT:R_Axial_DIN0207_L6.3mm_D2.5mm_P7.62mm_Horizontal -> incinerator:R_THT_D2.5mm_P7.62mm_Custom

Commit message: added traces & ground planes
Parts:
- J8: value To Rotary Encoder / Switch -> To Encoder
- J9: value Waveshare 4.2\" e-paper -> To Display
Connections:
- net ROT_CLK: now also U2.11 (D14); no longer U2.12 (D12)
- net ROT_DT: now also U2.12 (D12); no longer U2.11 (D14)
Changed lines of the file:
@@
 P 10350 3650
 F 0 "J9" H 10458 3117 50  0000 C CNN
-F 1 "Waveshare 4.2\" e-paper" H 10458 3026 50  0000 C CNN
+F 1 "To Display" H 10458 3026 50  0000 C CNN
 F 2 "Connector_PinHeader_2.54mm:PinHeader_1x08_P2.54mm_Vertical" H 10350 3650 50  0001 C CNN
 F 3 "~" H 10350 3650 50  0001 C CNN
@@
 	0    -1   1    0
 $EndComp
-Wire Wire Line
-	6750 4250 6050 4250
-Wire Wire Line
-	6050 4250 6050 4850
-Wire Wire Line
-	6750 4150 5900 4150
 $Comp
 L Device:Q_NMOS_GDS Q1
@@
 P 7250 5600
 F 0 "J8" V 7404 5844 50  0000 L CNN
-F 1 "To Rotary Encoder / Switch" V 7313 5844 50  0000 L CNN
+F 1 "To Encoder" V 7313 5844 50  0000 L CNN
 F 2 "Connector_PinHeader_2.54mm:PinHeader_1x05_P2.54mm_Vertical" H 7250 5600 50  0001 C CNN
 F 3 "~" H 7250 5600 50  0001 C CNN
@@
 Wire Wire Line
 	7250 4850 7250 5400
-Wire Wire Line
-	5900 5000 7050 5000
-Wire Wire Line
-	7050 5000 7050 5400
-Wire Wire Line
-	5900 4150 5900 5000
 Wire Wire Line
 	8600 4850 7350 4850
@@
 Wire Wire Line
 	5050 5050 5550 5050
+Wire Wire Line
+	6050 4150 6750 4150
+Wire Wire Line
+	6050 4150 6050 4850
+Wire Wire Line
+	6750 4250 6150 4250
+Wire Wire Line
+	6150 4250 6150 4950
+Wire Wire Line
+	6150 4950 7050 4950
+Wire Wire Line
+	7050 4950 7050 5400
 $EndSCHEMATC
